File: HagiwoBuffMult.kicad_sch (KiCad schematic)
At the start: 43 parts, among them J10 Conn_01x01_Pin, J11 Conn_01x01_Pin, J12 Conn_01x01_Pin, J13 Conn_01x01_Pin, J14 Conn_01x01_Pin, J15 Conn_01x01_Pin, J16 Conn_01x01_Pin, J17 Conn_01x01_Socket, J18 Conn_01x01_Socket, J19 Conn_01x01_Socket, J20 Conn_01x01_Socket, J21 Conn_01x01_Socket, J22 Conn_01x01_Socket, J23 Conn_01x01_Socket, J24 Conn_01x01_Socket, J25 Conn_01x01_Socket, J26 Conn_01x01_Socket, J6 Conn_01x01_Pin, J7 Conn_01x01_Pin, J8 Conn_01x01_Pin, J9 Eurorack_Power_10pin_Unshroud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, U1 TL074, U2 TL074

Commit message: routed and made panel
Parts:
- removed C3, C4: 100n, Capacitor_THT:C_Axial_L3.8mm_D2.6mm_P7.50mm_Horizontal, symbol Device:C
- J1: renamed from IN1; value 3.5mm_Mono_Switched_sm -> IN1
- J2: renamed from IN2; value 3.5mm_Mono_Switched_sm -> IN2
- J4: renamed from OUT1; value 3.5mm_Mono_Switched_sm -> OUT1
- J5: renamed from OUT2; value 3.5mm_Mono_Switched_sm -> OUT2
- J6: renamed from OUT3; value 3.5mm_Mono_Switched_sm -> OUT3
- J7: renamed from OUT4; value 3.5mm_Mono_Switched_sm -> OUT4
- J8: renamed from OUT5; value 3.5mm_Mono_Switched_sm -> OUT5
- J9: renamed from OUT6; value 3.5mm_Mono_Switched_sm -> OUT6
- renumbered J17 to J10, J18 to J11, J19 to J12, J20 to J13, J21 to J14, J22 to J15, J23 to J16, J24 to J17, J25 to J18, J26 to J19, J6 to J20, J7 to J21, J8 to J22, J10 to J23, J11 to J24, J12 to J25, J13 to J26, J14 to J27, J15 to J28, J16 to J29, J9 to J3, R5 to R2, R2 to R3, R3 to R4, R4 to R5
Connections:
- net IN1_PIN1_C: no longer U2.3 (+)
- net IN2_PIN1_C: now also U2.3 (+)

Commit message: added branding and instructions
Parts:
- J3: footprint Library:IDC-Header_2x05_P2.54mm_Vertical_Euro_Power_Striped -> Library:IDC-Header_2x05_P2.54mm_Vertical_Euro_Power_Striped_ThickerText
Changed lines of the file:
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@@
 			)
 		)
-		(property "Footprint" "Library:IDC-Header_2x05_P2.54mm_Vertical_Euro_Power_Striped"
+		(property "Footprint" "Library:IDC-Header_2x05_P2.54mm_Vertical_Euro_Power_Striped_ThickerText"
 			(at 39.37 157.48 0)
 			(effects

Commit message: v1.0 ready for production
Parts:
- C1, C2: value 10u -> 10uF; footprint Capacitor_THT:CP_Radial_D5.0mm_P2.50mm -> Capacitor_THT:CP_Radial_D4.0mm_P1.50mm; Silkscreen Value (none) -> 10uF▲
- J10, J11, J12, J13, J14, J15, J16, J17, J18, J19: Silkscreen Value (none) -> S
- J20, J21, J22, J23, J24, J25, J26, J27, J28, J29: Silkscreen Value (none) -> P
Other:
- note removed: "? x 2-pin sockets on front board ? x 2-pin sockets on back board 9 sockets total 8 for tip of each jack, 1 for ground of all jacks"
- note removed: "How does switched jack work? When not plugged then?"
Changed lines of the file:
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@@
 		)
 	)
-	(text "How does switched jack work? When not plugged then?"
-		(exclude_from_sim no)
-		(at 137.668 147.574 0)
-		(effects
-			(font
-				(size 1.27 1.27)
-			)
-		)
-	)
-	(text "? x 2-pin sockets on front board\n? x 2-pin sockets on back board\n\n9 sockets total\n8 for tip of each jack, 1 for ground of all jacks"
-		(exclude_from_sim no)
-		(at 110.744 139.446 0)
-		(effects
-			(font
-				(size 1.27 1.27)
-			)
-			(justify left)
-		)
-	)
 	(text "Front board"
 		(exclude_from_sim no)
@@
 			)
 		)
+		(property "Silkscreen Value" "P"
+			(at 257.81 72.39 0)
+			(effects
+				(font
+					(size 1.27 1.27)
+				)
+				(hide yes)
+			)
+		)
 		(pin "1"
 		)
@@
 			)
 		)
+		(property "Silkscreen Value" "S"
+			(at 208.28 82.55 0)
+			(effects
+				(font
+					(size 1.27 1.27)
+				)
+				(hide yes)
+			)
+		)
 		(pin "1"
 		)
@@
 			)
 		)
+		(property "Silkscreen Value" "S"
+			(at 208.28 72.39 0)
+			(effects
+				(font
+					(size 1.27 1.27)
+				)
+				(hide yes)
+			)
+		)
 		(pin "1"
 		)
@@
 			)
 		)
-		(property "Value" "10u"
+		(property "Value" "10uF"
 			(at 52.07 143.8909 0)
 			(effects
@@
 			)
 		)
-		(property "Footprint" "Capacitor_THT:CP_Radial_D5.0mm_P2.50mm"
+		(property "Footprint" "Capacitor_THT:CP_Radial_D4.0mm_P1.50mm"
 			(at 49.2252 147.32 0)
 			(effects
@@
 			)
 		)
+		(property "Silkscreen Value" "10uF▲"
+			(at 48.26 143.51 0)
+			(effects
+				(font
+					(size 1.27 1.27)
+				)
+				(hide yes)
+			)
+		)
 		(pin "1"
 		)
@@
 			)
 		)
+		(property "Silkscreen Value" "S"
+			(at 208.28 102.87 0)
+			(effects
+				(font
+					(size 1.27 1.27)
+				)
+				(hide yes)
+			)
+		)
 		(pin "1"
 		)
@@
 			)
 		)
+		(property "Silkscreen Value" "P"
+			(at 257.81 74.93 0)
+			(effects
+				(font
+					(size 1.27 1.27)
+				)
+				(hide yes)
+			)
+		)
 		(pin "1"
 		)
@@
 			)
 		)
+		(property "Silkscreen Value" "P"
+			(at 257.81 90.17 0)
+			(effects
+				(font
+					(size 1.27 1.27)
+				)
+				(hide yes)
+			)
+		)
 		(pin "1"
 		)
@@
 			)
 		)
+		(property "Silkscreen Value" "S"
+			(at 208.28 80.01 0)
+			(effects
+				(font
+					(size 1.27 1.27)
+				)
+				(hide yes)
+			)
+		)
 		(pin "1"
 		)
@@
 			)
 		)
+		(property "Silkscreen Value" "P"
+			(at 257.81 80.01 0)
+			(effects
+				(font
+					(size 1.27 1.27)
+				)
+				(hide yes)
+			)
+		)
 		(pin "1"
 		)
@@
 			)
 		)
+		(property "Silkscreen Value" "S"
+			(at 208.28 90.17 0)
+			(effects
+				(font
+					(size 1.27 1.27)
+				)
+				(hide yes)
+			)
+		)
 		(pin "1"
 		)
@@
 			)
 		)
+		(property "Silkscreen Value" "P"
+			(at 257.81 102.87 0)
+			(effects
+				(font
+					(size 1.27 1.27)
+				)
+				(hide yes)
+			)
+		)
 		(pin "1"
 		)
@@
 			)
 		)
+		(property "Silkscreen Value" "S"
+			(at 208.28 74.93 0)
+			(effects
+				(font
+					(size 1.27 1.27)
+				)
+				(hide yes)
+			)
+		)
 		(pin "1"
 		)
@@
 			)
 		)
+		(property "Silkscreen Value" "S"
+			(at 208.28 87.63 0)
+			(effects
+				(font
+					(size 1.27 1.27)
+				)
+				(hide yes)
+			)
+		)
 		(pin "1"
 		)
@@
 			)
 		)
+		(property "Silkscreen Value" "S"
+			(at 208.28 95.25 0)
+			(effects
+				(font
+					(size 1.27 1.27)
+				)
+				(hide yes)
+			)
+		)
 		(pin "1"
 		)
@@
 			)
 		)
+		(property "Silkscreen Value" "P"
+			(at 257.81 97.79 0)
+			(effects
+				(font
+					(size 1.27 1.27)
+				)
+				(hide yes)
+			)
+		)
 		(pin "1"
 		)
@@
 			)
 		)
+		(property "Silkscreen Value" "S"
+			(at 208.28 105.41 0)
+			(effects
+				(font
+					(size 1.27 1.27)
+				)
+				(hide yes)
+			)
+		)
 		(pin "1"
 		)
@@
 			)
 		)
-		(property "Value" "10u"
+		(property "Value" "10uF"
 			(at 52.07 151.5109 0)
 			(effects
@@
 			)
 		)
-		(property "Footprint" "Capacitor_THT:CP_Radial_D5.0mm_P2.50mm"
+		(property "Footprint" "Capacitor_THT:CP_Radial_D4.0mm_P1.50mm"
 			(at 49.2252 154.94 0)
 			(effects
@@
 			)
 		)
+		(property "Silkscreen Value" "10uF▲"
+			(at 48.26 151.13 0)
+			(effects
+				(font
+					(size 1.27 1.27)
+				)
+				(hide yes)
+			)
+		)
 		(pin "1"
 		)
@@
 			)
 		)
+		(property "Silkscreen Value" "S"
+			(at 208.28 97.79 0)
+			(effects
+				(font
+					(size 1.27 1.27)
+				)
+				(hide yes)
+			)
+		)
 		(pin "1"
 		)
@@
 			)
 		)
+		(property "Silkscreen Value" "P"
+			(at 257.81 87.63 0)
+			(effects
+				(font
+					(size 1.27 1.27)
+				)
+				(hide yes)
+			)
+		)
 		(pin "1"
 		)
@@
 			)
 		)
+		(property "Silkscreen Value" "P"
+			(at 257.81 105.41 0)
+			(effects
+				(font
+					(size 1.27 1.27)
+				)
+				(hide yes)
+			)
+		)
 		(pin "1"
 		)
@@
 			)
 		)
+		(property "Silkscreen Value" "P"
+			(at 257.81 95.25 0)
+			(effects
+				(font
+					(size 1.27 1.27)
+				)
+				(hide yes)
+			)
+		)
 		(pin "1"
 		)
@@
 			(at 257.81 82.55 0)
 			(effects
+				(font
+					(size 1.27 1.27)
+				)
+				(hide yes)
+			)
+		)
+		(property "Silkscreen Value" "P"
+			(at 257.81 82.55 0)
+			(effects

Commit message: working on v1.1 - added build notes - widened 10uF cap footprint - what to do about traces being too close to board edge?
Parts:
- C1, C2: footprint Capacitor_THT:CP_Radial_D4.0mm_P1.50mm -> Capacitor_THT:CP_Radial_D4.0mm_P2.00mm
Changed lines of the file:
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@@
 			)
 		)
-		(property "Footprint" "Capacitor_THT:CP_Radial_D4.0mm_P1.50mm"
+		(property "Footprint" "Capacitor_THT:CP_Radial_D4.0mm_P2.00mm"
 			(at 49.2252 147.32 0)
 			(effects
@@
 			)
 		)
-		(property "Footprint" "Capacitor_THT:CP_Radial_D4.0mm_P1.50mm"
+		(property "Footprint" "Capacitor_THT:CP_Radial_D4.0mm_P2.00mm"
 			(at 49.2252 154.94 0)
 			(effects

Commit message: v1.1 reaady for final check
Parts:
- added C3, C4, C5, C6: 100nF, Capacitor_THT:C_Disc_D3.0mm_W1.6mm_P2.50mm, symbol Device:C
- R1: footprint Resistor_THT:R_Axial_DIN0207_L6.3mm_D2.5mm_P7.62mm_Horizontal -> Resistor_THT:R_Axial_DIN0204_L3.6mm_D1.6mm_P1.90mm_Vertical; Silkscreen Value (none) -> ▼330
- R2, R6, R8: footprint Resistor_THT:R_Axial_DIN0207_L6.3mm_D2.5mm_P7.62mm_Horizontal -> Resistor_THT:R_Axial_DIN0204_L3.6mm_D1.6mm_P1.90mm_Vertical; Silkscreen Value (none) -> 330▶
- R3, R4, R5, R7: footprint Resistor_THT:R_Axial_DIN0207_L6.3mm_D2.5mm_P7.62mm_Horizontal -> Resistor_THT:R_Axial_DIN0204_L3.6mm_D1.6mm_P1.90mm_Vertical; Silkscreen Value (none) -> ◀330
Connections:
- net +12V: now also C3.1, C4.1
- net -12V: now also C5.2, C6.2
- net GND: now also C3.2, C4.2, C5.1, C6.1
Other:
- moved on the sheet: U1E, U2E
